File: PCB/Revision 2/cpu.kicad_sch (KiCad schematic)
At the start: 38 parts, among them X1 CXO_SMD4, X2 32KHz

Commit message: Work on the schematic continutes
Parts:
- removed R10, R11, R12, R13, R14, R15, R16, R17, R18, R19, R3, R4, R5, R6, R7, R8, R9: 10KΩ, symbol Turaco:R
- added RN1, RN2, RN3, RN4, RN5: 10KΩ, symbol Device:R_Pack04_Split
- X2: value 32KHz -> 32.768kHz
Connections:
- net GND: now also RN3.4 (R4.1)
- net VCC: now also RN1.5 (R4.2), RN1.6 (R3.2), RN1.7 (R2.2), RN1.8 (R1.2), RN2.5 (R4.2), RN2.6 (R3.2), RN2.7 (R2.2), RN2.8 (R1.2), RN3.1 (R1.1), RN3.2 (R2.1), RN3.3 (R3.1), RN4.1 (R1.1), RN4.2 (R2.1), RN4.3 (R3.1), RN4.4 (R4.1), RN5.1 (R1.1), RN5.2 (R2.1), RN5.3 (R3.1), RN5.4 (R4.1)
- net ~{BUSACK}: now also RN5.7 (R2.2)
- net ~{BUSRQ}: now also RN5.6 (R3.2)
- net ~{CS0}: now also RN4.7 (R2.2)
- net ~{CS1}: now also RN4.6 (R3.2)
- net ~{CS2}: now also RN4.5 (R4.2)
- net ~{CS3}: now also RN3.8 (R1.2)
- net ~{FPGA_RESET}: now also RN3.5 (R4.2)
- net ~{IORQ}: now also RN2.4 (R4.1)
- net ~{IRQ0}: now also RN3.7 (R2.2)
- net ~{IRQ1}: now also RN3.6 (R3.2)
- net ~{MREQ}: now also RN2.3 (R3.1)
- net ~{NMI}: now also RN5.5 (R4.2)
- net ~{RD}: now also RN2.2 (R2.1)
- net ~{RESET}: now also RN4.8 (R1.2)
- net ~{SS1}: now also RN1.3 (R3.1)
- net ~{SS2}: now also RN1.2 (R2.1)
- net ~{SS3}: now also RN1.1 (R1.1)
- net ~{WAIT}: now also RN5.8 (R1.2)
- net ~{WP}: now also RN1.4 (R4.1)
- net ~{WR}: now also RN2.1 (R1.1)
- net PHI: now reaches U2.111 (PHI)
- no-connect marks 12 -> 11
