File: PCB/Revision 2/cpu.kicad_sch (KiCad schematic)
At the start: 26 parts, among them X1 CXO_SMD4, X2 32.768kHz

Commit message: Updated re: issue #2
Parts:
- added R3: 10Ω, symbol Device:R
- C10, C11, C12, C13, C14, C15, C16, C17, C18, C19, C3, C4, C5, C59, C6, C7, C8, C9: footprint (none) -> Capacitor_SMD:C_0402_1005Metric
- RN1, RN2, RN3, RN4, RN5: footprint (none) -> Resistor_SMD:R_Array_Concave_4x0402
Connections:
- net MOSI: now also R3.1; no longer U2.107 (PB7•MOSI)
- new net: R3.2, U2.107 (PB7•MOSI)
Other:
- moved on the sheet: C18, C19, U2I, X2
