File: PCB/Revision 2/dvi_transmitter.kicad_sch (KiCad schematic)
At the start: 28 parts, among them U5 TFP410PAP

Commit message: Work on the schematic continutes
Parts:
- removed R20, R21, R22, R23, R24, R25: 10KΩ, symbol Turaco:R
- added RN2 (x2): 10KΩ, symbol Device:R_Pack04_Split
Connections:
- net GND: now also RN2.7 (R2.2), RN2.8 (R1.2)
- net VCC: now also RN2.1 (R1.1), RN2.2 (R2.1), RN2.3 (R3.1), RN2.4 (R4.1)
- net at JP2.1 (A), U5.35 (DKEN): now also RN2.7 (R2.2)
- net at U5.14 (DSEL/SDA): now also RN2.1 (R1.1)
- net at U5.10 (~PD): now also RN2.6 (R3.2)
- net at U5.9 (EDGE/HTPLG): now also RN2.8 (R1.2)
- net at U5.15 (BSEL/SCL): now also RN2.5 (R4.2)
- net at U5.13 (ISEL/~RST): now also RN2.2 (R2.1)
