File: PCB/Revision 2/dvi_transmitter.kicad_sch (KiCad schematic)
At the start: 24 parts, among them U5 TFP410PAP

Commit message: Updated re: issue #2
Parts:
- C22, C23, C24, C25, C26, C27, C28, C29, C30, C31, C32, C33: footprint (none) -> Capacitor_SMD:C_0402_1005Metric
- JP1, JP3, JP4: footprint (none) -> Jumper:SolderJumper-3_P1.3mm_Bridged12_Pad1.0x1.5mm
- JP2: footprint (none) -> Jumper:SolderJumper-2_P1.3mm_Open_Pad1.0x1.5mm
- L1, L2, L3: footprint (none) -> Inductor_SMD:L_0603_1608Metric
- RN2: footprint (none) -> Resistor_SMD:R_Array_Concave_4x0402
Changed lines of the file:
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@@
       (effects (font (size 1.27 1.27)) (justify left))
     )
-    (property "Footprint" "" (at 220.6752 106.68 0)
+    (property "Footprint" "Capacitor_SMD:C_0402_1005Metric" (at 220.6752 106.68 0)
       (effects (font (size 1.27 1.27)) hide)
     )
@@
       (effects (font (size 1.27 1.27)) (justify left) hide)
     )
-    (property "Footprint" "" (at 90.17 158.75 0)
+    (property "Footprint" "Jumper:SolderJumper-2_P1.3mm_Open_Pad1.0x1.5mm" (at 90.17 158.75 0)
       (effects (font (size 1.27 1.27)) hide)
     )
@@
       (effects (font (size 1.27 1.27)) (justify left))
     )
-    (property "Footprint" "" (at 220.6752 63.5 0)
+    (property "Footprint" "Capacitor_SMD:C_0402_1005Metric" (at 220.6752 63.5 0)
       (effects (font (size 1.27 1.27)) hide)
     )
@@
       (effects (font (size 1.27 1.27)) (justify left))
     )
-    (property "Footprint" "" (at 235.9152 85.09 0)
+    (property "Footprint" "Capacitor_SMD:C_0402_1005Metric" (at 235.9152 85.09 0)
       (effects (font (size 1.27 1.27)) hide)
     )
@@
       (effects (font (size 1.27 1.27)) (justify left))
     )
-    (property "Footprint" "" (at 235.9152 63.5 0)
+    (property "Footprint" "Capacitor_SMD:C_0402_1005Metric" (at 235.9152 63.5 0)
       (effects (font (size 1.27 1.27)) hide)
     )
@@
       (effects (font (size 1.27 1.27)))
     )
-    (property "Footprint" "" (at 127.762 153.67 90)
+    (property "Footprint" "Resistor_SMD:R_Array_Concave_4x0402" (at 127.762 153.67 90)
       (effects (font (size 1.27 1.27)) hide)
     )
@@
       (effects (font (size 1.27 1.27)))
     )
-    (property "Footprint" "" (at 241.3 74.93 0)
+    (property "Footprint" "Inductor_SMD:L_0603_1608Metric" (at 241.3 74.93 0)
       (effects (font (size 1.27 1.27)) hide)
     )
@@
       (effects (font (size 1.27 1.27)) (justify left) hide)
     )
-    (property "Footprint" "" (at 82.55 158.75 0)
+    (property "Footprint" "Jumper:SolderJumper-3_P1.3mm_Bridged12_Pad1.0x1.5mm" (at 82.55 158.75 0)
       (effects (font (size 1.27 1.27)) hide)
     )
@@
       (effects (font (size 1.27 1.27)) (justify left))
     )
-    (property "Footprint" "" (at 235.9152 106.68 0)
+    (property "Footprint" "Capacitor_SMD:C_0402_1005Metric" (at 235.9152 106.68 0)
       (effects (font (size 1.27 1.27)) hide)
     )
@@
       (effects (font (size 1.27 1.27)) (justify left))
     )
-    (property "Footprint" "" (at 228.2952 63.5 0)
+    (property "Footprint" "Capacitor_SMD:C_0402_1005Metric" (at 228.2952 63.5 0)
       (effects (font (size 1.27 1.27)) hide)
     )
@@
       (effects (font (size 1.27 1.27)) (justify left))
     )
-    (property "Footprint" "" (at 213.0552 85.09 0)
+    (property "Footprint" "Capacitor_SMD:C_0402_1005Metric" (at 213.0552 85.09 0)
       (effects (font (size 1.27 1.27)) hide)
     )
@@
       (effects (font (size 1.27 1.27)))
     )
-    (property "Footprint" "" (at 241.3 96.52 0)
+    (property "Footprint" "Inductor_SMD:L_0603_1608Metric" (at 241.3 96.52 0)
       (effects (font (size 1.27 1.27)) hide)
     )
@@
       (effects (font (size 1.27 1.27)) (justify left) hide)
     )
-    (property "Footprint" "" (at 97.79 158.75 0)
+    (property "Footprint" "Jumper:SolderJumper-3_P1.3mm_Bridged12_Pad1.0x1.5mm" (at 97.79 158.75 0)
       (effects (font (size 1.27 1.27)) hide)
     )
@@
       (effects (font (size 1.27 1.27)) (justify left))
     )
-    (property "Footprint" "" (at 220.6752 85.09 0)
+    (property "Footprint" "Capacitor_SMD:C_0402_1005Metric" (at 220.6752 85.09 0)
       (effects (font (size 1.27 1.27)) hide)
     )
@@
       (effects (font (size 1.27 1.27)))
     )
-    (property "Footprint" "" (at 83.312 113.03 90)
+    (property "Footprint" "Resistor_SMD:R_Array_Concave_4x0402" (at 83.312 113.03 90)
       (effects (font (size 1.27 1.27)) hide)
     )
@@
       (effects (font (size 1.27 1.27)))
     )
-    (property "Footprint" "" (at 74.422 113.03 90)
+    (property "Footprint" "Resistor_SMD:R_Array_Concave_4x0402" (at 74.422 113.03 90)
       (effects (font (size 1.27 1.27)) hide)
     )
@@
       (effects (font (size 1.27 1.27)) (justify left) hide)
     )
-    (property "Footprint" "" (at 107.95 158.75 0)
+    (property "Footprint" "Jumper:SolderJumper-3_P1.3mm_Bridged12_Pad1.0x1.5mm" (at 107.95 158.75 0)
       (effects (font (size 1.27 1.27)) hide)
     )
@@
       (effects (font (size 1.27 1.27)))
     )
-    (property "Footprint" "" (at 92.202 113.03 90)
+    (property "Footprint" "Resistor_SMD:R_Array_Concave_4x0402" (at 92.202 113.03 90)
       (effects (font (size 1.27 1.27)) hide)
     )
@@
       (effects (font (size 1.27 1.27)))
     )
-    (property "Footprint" "" (at 118.872 153.67 90)
+    (property "Footprint" "Resistor_SMD:R_Array_Concave_4x0402" (at 118.872 153.67 90)
       (effects (font (size 1.27 1.27)) hide)
     )
@@
       (effects (font (size 1.27 1.27)) (justify left))
     )
-    (property "Footprint" "" (at 213.0552 63.5 0)
+    (property "Footprint" "Capacitor_SMD:C_0402_1005Metric" (at 213.0552 63.5 0)
       (effects (font (size 1.27 1.27)) hide)
     )
@@
       (effects (font (size 1.27 1.27)))
     )
-    (property "Footprint" "" (at 241.3 53.34 0)
+    (property "Footprint" "Inductor_SMD:L_0603_1608Metric" (at 241.3 53.34 0)
       (effects (font (size 1.27 1.27)) hide)
     )
@@
       (effects (font (size 1.27 1.27)) (justify left))
     )
-    (property "Footprint" "" (at 228.2952 85.09 0)
+    (property "Footprint" "Capacitor_SMD:C_0402_1005Metric" (at 228.2952 85.09 0)
       (effects (font (size 1.27 1.27)) hide)
     )
@@
       (effects (font (size 1.27 1.27)))
     )
-    (property "Footprint" "" (at 101.092 113.03 90)
+    (property "Footprint" "Resistor_SMD:R_Array_Concave_4x0402" (at 101.092 113.03 90)
       (effects (font (size 1.27 1.27)) hide)
     )
@@
       (effects (font (size 1.27 1.27)) (justify left))
     )
-    (property "Footprint" "" (at 213.0552 106.68 0)
+    (property "Footprint" "Capacitor_SMD:C_0402_1005Metric" (at 213.0552 106.68 0)
       (effects (font (size 1.27 1.27)) hide)
     )
@@
       (effects (font (size 1.27 1.27)) (justify left))
     )
-    (property "Footprint" "" (at 228.2952 106.68 0)
-      (effects (font (size 1.27 1.27)) hide)
-    )
+    (property "Footprint" "Capacitor_SMD:C_0402_1005Metric" (at 228.2952 106.68 0)
+      (effects (font (size 1.27 1.27)) hide)
+    )
