File: PCB/Revision 2/vera.kicad_sch (KiCad schematic)
At the start: 15 parts, among them U3 74CB3T1G125, U4 ICE40UP5K-SG48ITR50, X3 SG5032CAN_25.000000M-TJGA3

Commit message: Work on the schematic continutes
Parts:
- removed X3: SG5032CAN_25.000000M-TJGA3, symbol Turaco:SG-5032CAN
- added U11: 74LVC2G32, symbol 74xGxx:74LVC2G32
- C52, C55, C56: value 4.7uF -> 4.7µF
Connections:
- net CDONE: no longer U3.1 (~{OE})
- net DE: now also U4.32 (IOT_43A); no longer U3.4 (B), U4.14 (IOB_32A_SPI_SO)
- net GND: now also U11.4 (GND)
- net SYSCLK: now also U4.28 (IOT_41A); no longer U4.35 (IOT_46B_G0)
- net VCC: now also U11.8 (VCC)
- net ~{CS1}: now also U11.2, U11.6; no longer U4.28 (IOT_41A)
- net ~{IRQ0}: no longer U4.32 (IOT_43A)
- net ~{RD}: now also U11.1; no longer U4.36 (IOT_48B)
- net ~{SS1}: now also U3.1 (~{OE})
- net ~{WR}: now also U11.5; no longer U4.31 (IOT_42B)
- new net PHI: U4.35 (IOT_46B_G0)
- new net ~{CSRD}: U11.7, U4.36 (IOT_48B)
- new net ~{CSWR}: U11.3, U4.31 (IOT_42B)
- new net ~{IRQ1}: U3.4 (B), U4.14 (IOB_32A_SPI_SO)
- no-connect marks 1 -> 0
Other:
- note added: "The VERA bitstream has been altered; after bootloading, the MISO pin is reassigned to /IRQ1, the output which sends an interrupt to the CPU. The MISO signal is gated to that FPGA pin by a 74CB3T1G125 single FET switch, controlled by the SPI select signal of the FPGA. When that signal is high, the MISO line is isolated from the FPGA by the FET. The CPU must make sure to disable /IRQ1 before bootlo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"
- note removed: "The VERA bitstream has been altered; after bootloading, the MISO pin is reassigned to DE, the display enable output to control the DVI transmitter. The MISO signal is gated to that FPGA pin by a 74CB3T1G125 single FET switch, controlled by the FPGA's CDONE output. Once CDONE goes high, the MISO signal is isolated from the DE signal until the FPGA is rebooted and bootloaded."
- moved on the sheet: C20, C47, C48, C49, C50, C51, C52, C53, C54, C55, C56, U3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
