File: PCB/Revision 2/vera.kicad_sch (KiCad schematic)
At the start: 15 parts, among them U11 74LVC2G32, U3 74CB3T1G125, U4 ICE40UP5K-SG48ITR50

Commit message: Updated re: issue #2
Parts:
- C20, C21, C47, C48, C49, C50, C51, C52, C53, C54, C55, C56: footprint (none) -> Capacitor_SMD:C_0402_1005Metric
Changed lines of the file:
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@@
     (effects (font (size 1.27 1.27)) (justify left bottom))
   )
-  (label "PHI" (at 220.98 49.53 0)
+  (label "PHI" (at 220.98 49.53 0) (fields_autoplaced)
     (effects (font (size 1.27 1.27)) (justify left bottom))
   )
@@
       (effects (font (size 1.27 1.27)) (justify left))
     )
-    (property "Footprint" "" (at 165.1 138.43 0)
+    (property "Footprint" "Capacitor_SMD:C_0402_1005Metric" (at 165.1 138.43 0)
       (effects (font (size 1.27 1.27)) hide)
     )
@@
       (effects (font (size 1.27 1.27)) (justify left))
     )
-    (property "Footprint" "" (at 176.53 138.43 0)
+    (property "Footprint" "Capacitor_SMD:C_0402_1005Metric" (at 176.53 138.43 0)
       (effects (font (size 1.27 1.27)) hide)
     )
@@
   )
   (symbol (lib_id "Turaco:ICE40UP5K-SG48ITR50") (at 121.92 71.12 0) (unit 1)
-    (in_bom yes) (on_board yes) (dnp no) (fields_autoplaced)
-    (property "Reference" "U4" (at 138.43 66.04 0)
-      (effects (font (size 1.27 1.27)))
-    )
-    (property "Value" "ICE40UP5K-SG48ITR50" (at 138.43 68.58 0)
+    (in_bom yes) (on_board yes) (dnp no)
+    (property "Reference" "U4" (at 123.19 69.85 0)
+      (effects (font (size 1.27 1.27)))
+    )
+    (property "Value" "ICE40UP5K-SG48ITR50" (at 144.78 69.85 0)
       (effects (font (size 1.27 1.27)))
     )
@@
       (effects (font (size 1.27 1.27)) (justify left))
     )
-    (property "Footprint" "" (at 63.5 130.81 0)
+    (property "Footprint" "Capacitor_SMD:C_0402_1005Metric" (at 63.5 130.81 0)
       (effects (font (size 1.27 1.27)) hide)
     )
@@
       (effects (font (size 1.27 1.27)) (justify left))
     )
-    (property "Footprint" "" (at 210.82 123.19 0)
+    (property "Footprint" "Capacitor_SMD:C_0402_1005Metric" (at 210.82 123.19 0)
       (effects (font (size 1.27 1.27)) hide)
     )
@@
       (effects (font (size 1.27 1.27)) (justify left))
     )
-    (property "Footprint" "" (at 187.96 123.19 0)
+    (property "Footprint" "Capacitor_SMD:C_0402_1005Metric" (at 187.96 123.19 0)
       (effects (font (size 1.27 1.27)) hide)
     )
@@
       (effects (font (size 1.27 1.27)) (justify left))
     )
-    (property "Footprint" "" (at 165.1 123.19 0)
+    (property "Footprint" "Capacitor_SMD:C_0402_1005Metric" (at 165.1 123.19 0)
       (effects (font (size 1.27 1.27)) hide)
     )
@@
       (effects (font (size 1.27 1.27)) (justify left))
     )
-    (property "Footprint" "" (at 176.53 123.19 0)
+    (property "Footprint" "Capacitor_SMD:C_0402_1005Metric" (at 176.53 123.19 0)
       (effects (font (size 1.27 1.27)) hide)
     )
@@
       (effects (font (size 1.27 1.27)) (justify left))
     )
-    (property "Footprint" "" (at 19.05 182.88 0)
+    (property "Footprint" "Capacitor_SMD:C_0402_1005Metric" (at 19.05 182.88 0)
       (effects (font (size 1.27 1.27)) hide)
     )
@@
       (effects (font (size 1.27 1.27)) (justify left))
     )
-    (property "Footprint" "" (at 187.96 138.43 0)
+    (property "Footprint" "Capacitor_SMD:C_0402_1005Metric" (at 187.96 138.43 0)
       (effects (font (size 1.27 1.27)) hide)
     )
@@
       (effects (font (size 1.27 1.27)) (justify left))
     )
-    (property "Footprint" "" (at 220.98 123.19 0)
+    (property "Footprint" "Capacitor_SMD:C_0402_1005Metric" (at 220.98 123.19 0)
       (effects (font (size 1.27 1.27)) hide)
     )
@@
       (effects (font (size 1.27 1.27)) (justify left))
     )
-    (property "Footprint" "" (at 199.39 123.19 0)
+    (property "Footprint" "Capacitor_SMD:C_0402_1005Metric" (at 199.39 123.19 0)
       (effects (font (size 1.27 1.27)) hide)
     )
@@
       (effects (font (size 1.27 1.27)) (justify left))
     )
-    (property "Footprint" "" (at 199.39 138.43 0)
-      (effects (font (size 1.27 1.27)) hide)
-    )
+    (property "Footprint" "Capacitor_SMD:C_0402_1005Metric" (at 199.39 138.43 0)
+      (effects (font (size 1.27 1.27)) hide)
+    )
