File: PCB/Revision 2/Revision 2.kicad_sch (KiCad schematic)
At the start: 14 parts, among them J1 USB_C, U1 LD39150DT33, U10 AP3417CKTR-G1

Commit message: Updated re: issue #2
Parts:
- removed C1, C2: 10µF, symbol Turaco:C
- removed C57, C58: 10uF, symbol Turaco:C_Small
- added C1, C2, C57, C58: 10µF, symbol Device:C_Polarized
Connections:
- net +1V2: now also C57.1
- net +5V: now also C1.1
- net GND: now also C1.2, C2.2, C57.2, C58.2
- net VCC: now also C2.1
- net at R41.1, U10.1 (EN), U10.4 (VIN): now also C58.1
Changed lines of the file:
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@@
     (effects (font (size 1.27 1.27)) (justify left bottom))
   )
-  (symbol (lib_id "power:GND") (at 125.73 185.42 0) (unit 1)
-    (in_bom yes) (on_board yes) (dnp no)
-    (property "Reference" "#PWR0144" (at 125.73 191.77 0)
-      (effects (font (size 1.27 1.27)) hide)
-    )
-    (property "Value" "GND" (at 125.857 189.8142 0)
-      (effects (font (size 1.27 1.27)))
-    )
-    (property "Footprint" "" (at 125.73 185.42 0)
-      (effects (font (size 1.27 1.27)) hide)
-    )
-    (property "Datasheet" "" (at 125.73 185.42 0)
+  (symbol (lib_id "power:GND") (at 125.73 187.96 0) (unit 1)
+    (in_bom yes) (on_board yes) (dnp no)
+    (property "Reference" "#PWR0144" (at 125.73 194.31 0)
+      (effects (font (size 1.27 1.27)) hide)
+    )
+    (property "Value" "GND" (at 125.857 192.3542 0)
+      (effects (font (size 1.27 1.27)))
+    )
+    (property "Footprint" "" (at 125.73 187.96 0)
+      (effects (font (size 1.27 1.27)) hide)
+    )
+    (property "Datasheet" "" (at 125.73 187.96 0)
       (effects (font (size 1.27 1.27)) hide)
     )
@@
     )
   )
-  (symbol (lib_id "Turaco:C") (at 85.09 161.29 0) (unit 1)
-    (in_bom yes) (on_board yes) (dnp no)
-    (property "Reference" "C2" (at 86.36 158.7499 0)
-      (effects (font (size 1.27 1.27)) (justify left))
-    )
-    (property "Value" "10µF" (at 86.36 163.8299 0)
-      (effects (font (size 1.27 1.27)) (justify left))
-    )
-    (property "Footprint" "" (at 86.0552 165.1 0)
-      (effects (font (size 1.27 1.27)) hide)
-    )
-    (property "Datasheet" "~" (at 85.09 161.29 0)
-      (effects (font (size 1.27 1.27)) hide)
-    )
-    (pin "1")
-    (pin "2")
-    (instances
-      (project "Revision 2"
-        (path "/3ba39048-ccb5-49b6-bc29-f9a8dd2e53b6"
-          (reference "C2") (unit 1)
-        )
-      )
-    )
-  )
   (symbol (lib_id "power:PWR_FLAG") (at 25.4 185.42 90) (unit 1)
     (in_bom yes) (on_board yes) (dnp no)
@@
     )
   )
+  (symbol (lib_id "Device:C_Polarized") (at 64.77 161.29 0) (unit 1)
+    (in_bom yes) (on_board yes) (dnp no) (fields_autoplaced)
+    (property "Reference" "C1" (at 68.58 159.1309 0)
+      (effects (font (size 1.27 1.27)) (justify left))
+    )
+    (property "Value" "10µF" (at 68.58 161.6709 0)
+      (effects (font (size 1.27 1.27)) (justify left))
+    )
+    (property "Footprint" "" (at 65.7352 165.1 0)
+      (effects (font (size 1.27 1.27)) hide)
+    )
+    (property "Datasheet" "~" (at 64.77 161.29 0)
+      (effects (font (size 1.27 1.27)) hide)
+    )
+    (pin "1")
+    (pin "2")
+    (instances
+      (project "Revision 2"
+        (path "/3ba39048-ccb5-49b6-bc29-f9a8dd2e53b6"
+          (reference "C1") (unit 1)
+        )
+      )
+    )
+  )
   (symbol (lib_id "Turaco:R") (at 49.53 179.07 0) (unit 1)
     (in_bom yes) (on_board yes) (dnp no)
@@
     )
   )
-  (symbol (lib_id "power:GND") (at 78.74 185.42 0) (unit 1)
-    (in_bom yes) (on_board yes) (dnp no)
-    (property "Reference" "#PWR0146" (at 78.74 191.77 0)
-      (effects (font (size 1.27 1.27)) hide)
-    )
-    (property "Value" "GND" (at 78.867 189.8142 0)
-      (effects (font (size 1.27 1.27)))
-    )
-    (property "Footprint" "" (at 78.74 185.42 0)
-      (effects (font (size 1.27 1.27)) hide)
-    )
-    (property "Datasheet" "" (at 78.74 185.42 0)
+  (symbol (lib_id "Device:C_Polarized") (at 78.74 184.15 0) (unit 1)
+    (in_bom yes) (on_board yes) (dnp no)
+    (property "Reference" "C58" (at 80.01 181.9909 0)
+      (effects (font (size 1.27 1.27)) (justify left))
+    )
+    (property "Value" "10µF" (at 80.01 187.0709 0)
+      (effects (font (size 1.27 1.27)) (justify left))
+    )
+    (property "Footprint" "" (at 79.7052 187.96 0)
+      (effects (font (size 1.27 1.27)) hide)
+    )
+    (property "Datasheet" "~" (at 78.74 184.15 0)
+      (effects (font (size 1.27 1.27)) hide)
+    )
+    (pin "1")
+    (pin "2")
+    (instances
+      (project "Revision 2"
+        (path "/3ba39048-ccb5-49b6-bc29-f9a8dd2e53b6"
+          (reference "C58") (unit 1)
+        )
+      )
+    )
+  )
+  (symbol (lib_id "power:GND") (at 78.74 187.96 0) (unit 1)
+    (in_bom yes) (on_board yes) (dnp no)
+    (property "Reference" "#PWR0146" (at 78.74 194.31 0)
+      (effects (font (size 1.27 1.27)) hide)
+    )
+    (property "Value" "GND" (at 78.867 192.3542 0)
+      (effects (font (size 1.27 1.27)))
+    )
+    (property "Footprint" "" (at 78.74 187.96 0)
+      (effects (font (size 1.27 1.27)) hide)
+    )
+    (property "Datasheet" "" (at 78.74 187.96 0)
       (effects (font (size 1.27 1.27)) hide)
     )
@@
     )
   )
-  (symbol (lib_id "Turaco:C_Small") (at 125.73 182.88 0) (unit 1)
-    (in_bom yes) (on_board yes) (dnp no)
-    (property "Reference" "C57" (at 128.0668 181.7116 0)
-      (effects (font (size 1.27 1.27)) (justify left))
-    )
-    (property "Value" "10uF" (at 128.0668 184.023 0)
-      (effects (font (size 1.27 1.27)) (justify left))
-    )
-    (property "Footprint" "" (at 125.73 182.88 0)
-      (effects (font (size 1.27 1.27)) hide)
-    )
-    (property "Datasheet" "~" (at 125.73 182.88 0)
+  (symbol (lib_id "Device:C_Polarized") (at 125.73 184.15 0) (unit 1)
+    (in_bom yes) (on_board yes) (dnp no) (fields_autoplaced)
+    (property "Reference" "C57" (at 129.54 181.9909 0)
+      (effects (font (size 1.27 1.27)) (justify left))
+    )
+    (property "Value" "10µF" (at 129.54 184.5309 0)
+      (effects (font (size 1.27 1.27)) (justify left))
+    )
+    (property "Footprint" "" (at 126.6952 187.96 0)
+      (effects (font (size 1.27 1.27)) hide)
+    )
+    (property "Datasheet" "~" (at 125.73 184.15 0)
       (effects (font (size 1.27 1.27)) hide)
     )
@@
         )
       )
-      (project "vera-module-rev4"
-        (path "/718de4b0-0236-4070-9598-e8fe323a1b0b"
-          (reference "C24") (unit 1)
-        )
-      )
-    )
-  )
-  (symbol (lib_id "Turaco:C") (at 64.77 161.29 0) (unit 1)
-    (in_bom yes) (on_board yes) (dnp no)
-    (property "Reference" "C1" (at 66.04 158.7499 0)
-      (effects (font (size 1.27 1.27)) (justify left))
-    )
-    (property "Value" "10µF" (at 66.04 163.8299 0)
-      (effects (font (size 1.27 1.27)) (justify left))
-    )
-    (property "Footprint" "" (at 65.7352 165.1 0)
-      (effects (font (size 1.27 1.27)) hide)
-    )
-    (property "Datasheet" "~" (at 64.77 161.29 0)
-      (effects (font (size 1.27 1.27)) hide)
-    )
-    (pin "1")
-    (pin "2")
-    (instances
-      (project "Revision 2"
-        (path "/3ba39048-ccb5-49b6-bc29-f9a8dd2e53b6"
-          (reference "C1") (unit 1)
-        )
-      )
     )
   )
@@
         (path "/3ba39048-ccb5-49b6-bc29-f9a8dd2e53b6"
           (reference "#PWR05") (unit 1)
-        )
-      )
-    )
-  )
-  (symbol (lib_id "Turaco:C_Small") (at 78.74 182.88 0) (unit 1)
-    (in_bom yes) (on_board yes) (dnp no)
-    (property "Reference" "C58" (at 81.0768 181.7116 0)
-      (effects (font (size 1.27 1.27)) (justify left))
-    )
-    (property "Value" "10uF" (at 81.0768 184.023 0)
-      (effects (font (size 1.27 1.27)) (justify left))
-    )
-    (property "Footprint" "" (at 78.74 182.88 0)
-      (effects (font (size 1.27 1.27)) hide)
-    )
-    (property "Datasheet" "~" (at 78.74 182.88 0)
-      (effects (font (size 1.27 1.27)) hide)
-    )
-    (pin "1")
-    (pin "2")
-    (instances
-      (project "Revision 2"
-        (path "/3ba39048-ccb5-49b6-bc29-f9a8dd2e53b6"
-          (reference "C58") (unit 1)
-        )
-      )
-      (project "vera-module-rev4"
-        (path "/718de4b0-0236-4070-9598-e8fe323a1b0b"
-          (reference "C23") (unit 1)
         )
       )
@@
         )
       )
+    )
+  )
+  (symbol (lib_id "Device:C_Polarized") (at 85.09 161.29 0) (unit 1)
+    (in_bom yes) (on_board yes) (dnp no) (fields_autoplaced)
+    (property "Reference" "C2" (at 88.9 159.1309 0)
+      (effects (font (size 1.27 1.27)) (justify left))
+    )
+    (property "Value" "10µF" (at 88.9 161.6709 0)
+      (effects (font (size 1.27 1.27)) (justify left))
+    )
+    (property "Footprint" "" (at 86.0552 165.1 0)
+      (effects (font (size 1.27 1.27)) hide)
+    )
+    (property "Datasheet" "~" (at 85.09 161.29 0)
+      (effects (font (size 1.27 1.27)) hide)
+    )
+    (pin "1")
+    (pin "2")
+    (instances
+      (project "Revision 2"
+        (path "/3ba39048-ccb5-49b6-bc29-f9a8dd2e53b6"
+          (reference "C2") (unit 1)
+        )
+      )
