File: PCB/Revision 2/ethernet_header.kicad_sch (KiCad schematic)
At the start: 1 part, among them J4 Conn_02x10_Odd_Even

Commit message: Work on the schematic continutes
Parts:
- added RN2: 10KΩ, symbol Device:R_Pack04_Split
Connections:
- net ETH_COL: now also RN2.3 (R3.1)
- net ETH_CRS: now also RN2.1 (R1.1)
- net ETH_RX_CLK: now also RN2.2 (R2.1)
- net ETH_TX_CLK: now also RN2.4 (R4.1)
- net GND: now also RN2.5 (R4.2), RN2.6 (R3.2), RN2.7 (R2.2), RN2.8 (R1.2)
Changed lines of the file:
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@@
 (kicad_sch (version 20230121) (generator eeschema)
   (paper "USLetter")
+  (junction (at 191.77 92.71) (diameter 0) (color 0 0 0 0)
+  )
+  (junction (at 191.77 87.63) (diameter 0) (color 0 0 0 0)
+  )
+  (junction (at 191.77 97.79) (diameter 0) (color 0 0 0 0)
+  )
   (bus_entry (at 121.92 90.17) (size 2.54 2.54)
     (stroke (width 0) (type default))
@@
     (stroke (width 0) (type default))
   )
+  (bus_entry (at 165.1 95.25) (size 2.54 -2.54)
+    (stroke (width 0) (type default))
+  )
   (bus_entry (at 121.92 97.79) (size 2.54 2.54)
     (stroke (width 0) (type default))
   )
+  (bus_entry (at 165.1 85.09) (size 2.54 -2.54)
+    (stroke (width 0) (type default))
+  )
+  (bus_entry (at 165.1 90.17) (size 2.54 -2.54)
+    (stroke (width 0) (type default))
+  )
   (bus_entry (at 121.92 82.55) (size 2.54 2.54)
     (stroke (width 0) (type default))
@@
     (stroke (width 0) (type default))
   )
+  (bus_entry (at 165.1 100.33) (size 2.54 -2.54)
+    (stroke (width 0) (type default))
+  )
   (bus_entry (at 165.1 85.09) (size -2.54 -2.54)
     (stroke (width 0) (type default))
@@
     (stroke (width 0) (type default))
   )
+  (wire (pts (xy 191.77 82.55) (xy 191.77 87.63))
+    (stroke (width 0) (type default))
+  )
   (bus (pts (xy 165.1 97.79) (xy 165.1 100.33))
     (stroke (width 0) (type default))
   )
+  (wire (pts (xy 167.64 92.71) (xy 181.61 92.71))
+    (stroke (width 0) (type default))
+  )
+  (wire (pts (xy 189.23 92.71) (xy 191.77 92.71))
+    (stroke (width 0) (type default))
+  )
   (wire (pts (xy 152.4 105.41) (xy 149.86 105.41))
     (stroke (width 0) (type default))
@@
     (stroke (width 0) (type default))
   )
+  (wire (pts (xy 189.23 87.63) (xy 191.77 87.63))
+    (stroke (width 0) (type default))
+  )
   (wire (pts (xy 162.56 92.71) (xy 149.86 92.71))
     (stroke (width 0) (type default))
   )
+  (wire (pts (xy 191.77 87.63) (xy 191.77 92.71))
+    (stroke (width 0) (type default))
+  )
   (wire (pts (xy 124.46 90.17) (xy 137.16 90.17))
     (stroke (width 0) (type default))
   )
+  (wire (pts (xy 167.64 97.79) (xy 181.61 97.79))
+    (stroke (width 0) (type default))
+  )
   (wire (pts (xy 162.56 100.33) (xy 149.86 100.33))
     (stroke (width 0) (type default))
@@
     (stroke (width 0) (type default))
   )
+  (wire (pts (xy 189.23 82.55) (xy 191.77 82.55))
+    (stroke (width 0) (type default))
+  )
   (wire (pts (xy 124.46 92.71) (xy 137.16 92.71))
     (stroke (width 0) (type default))
@@
     (stroke (width 0) (type default))
   )
+  (wire (pts (xy 191.77 97.79) (xy 191.77 100.33))
+    (stroke (width 0) (type default))
+  )
   (bus (pts (xy 121.92 92.71) (xy 121.92 95.25))
     (stroke (width 0) (type default))
@@
     (stroke (width 0) (type default))
   )
+  (wire (pts (xy 167.64 82.55) (xy 181.61 82.55))
+    (stroke (width 0) (type default))
+  )
+  (wire (pts (xy 189.23 97.79) (xy 191.77 97.79))
+    (stroke (width 0) (type default))
+  )
+  (wire (pts (xy 167.64 87.63) (xy 181.61 87.63))
+    (stroke (width 0) (type default))
+  )
   (wire (pts (xy 124.46 97.79) (xy 137.16 97.79))
     (stroke (width 0) (type default))
@@
     (stroke (width 0) (type default))
   )
+  (wire (pts (xy 191.77 92.71) (xy 191.77 97.79))
+    (stroke (width 0) (type default))
+  )
   (wire (pts (xy 124.46 105.41) (xy 137.16 105.41))
     (stroke (width 0) (type default))
@@
     (effects (font (size 1.27 1.27)) (justify right bottom))
   )
+  (label "ETH_RX_CLK" (at 181.61 87.63 180)
+    (effects (font (size 1.27 1.27)) (justify right bottom))
+  )
   (label "ETH_RX_CLK" (at 137.16 90.17 180) (fields_autoplaced)
     (effects (font (size 1.27 1.27)) (justify right bottom))
@@
     (effects (font (size 1.27 1.27)) (justify right bottom))
   )
+  (label "ETH_COL" (at 181.61 92.71 180)
+    (effects (font (size 1.27 1.27)) (justify right bottom))
+  )
   (label "ETH_RX_ER" (at 137.16 87.63 180) (fields_autoplaced)
     (effects (font (size 1.27 1.27)) (justify right bottom))
@@
   (label "ETH_TXD1" (at 149.86 97.79 0) (fields_autoplaced)
     (effects (font (size 1.27 1.27)) (justify left bottom))
+  )
+  (label "ETH_CRS" (at 181.61 82.55 180)
+    (effects (font (size 1.27 1.27)) (justify right bottom))
+  )
+  (label "ETH_TX_CLK" (at 181.61 97.79 180)
+    (effects (font (size 1.27 1.27)) (justify right bottom))
   )
   (label "ETH_RXD1" (at 137.16 97.79 180) (fields_autoplaced)
@@
     )
   )
+  (symbol (lib_id "Device:R_Pack04_Split") (at 185.42 92.71 270) (unit 3)
+    (in_bom yes) (on_board yes) (dnp no)
+    (property "Reference" "RN2" (at 185.3757 90.8279 90)
+      (effects (font (size 1.27 1.27)))
+    )
+    (property "Value" "10KΩ" (at 185.42 92.71 90)
+      (effects (font (size 1.27 1.27)))
+    )
+    (property "Footprint" "" (at 185.42 90.678 90)
+      (effects (font (size 1.27 1.27)) hide)
+    )
+    (property "Datasheet" "~" (at 185.42 92.71 0)
+      (effects (font (size 1.27 1.27)) hide)
+    )
+    (pin "1")
+    (pin "8")
+    (pin "2")
+    (pin "7")
+    (pin "3")
+    (pin "6")
+    (pin "4")
+    (pin "5")
+    (instances
+      (project "Revision 2"
+        (path "/3ba39048-ccb5-49b6-bc29-f9a8dd2e53b6/e0049583-c97a-4b82-a4d7-59c894eac2f8"
+          (reference "RN2") (unit 3)
+        )
+        (path "/3ba39048-ccb5-49b6-bc29-f9a8dd2e53b6/b80782fd-1148-4a3e-8af5-19affa7e1aa8"
+          (reference "RN8") (unit 3)
+        )
+      )
+    )
+  )
+  (symbol (lib_id "Device:R_Pack04_Split") (at 185.42 97.79 270) (unit 4)
+    (in_bom yes) (on_board yes) (dnp no)
+    (property "Reference" "RN2" (at 185.3384 95.9414 90)
+      (effects (font (size 1.27 1.27)))
+    )
+    (property "Value" "10KΩ" (at 185.42 97.79 90)
+      (effects (font (size 1.27 1.27)))
+    )
+    (property "Footprint" "" (at 185.42 95.758 90)
+      (effects (font (size 1.27 1.27)) hide)
+    )
+    (property "Datasheet" "~" (at 185.42 97.79 0)
+      (effects (font (size 1.27 1.27)) hide)
+    )
+    (pin "1")
+    (pin "8")
+    (pin "2")
+    (pin "7")
+    (pin "3")
+    (pin "6")
+    (pin "4")
+    (pin "5")
+    (instances
+      (project "Revision 2"
+        (path "/3ba39048-ccb5-49b6-bc29-f9a8dd2e53b6/e0049583-c97a-4b82-a4d7-59c894eac2f8"
+          (reference "RN2") (unit 4)
+        )
+        (path "/3ba39048-ccb5-49b6-bc29-f9a8dd2e53b6/b80782fd-1148-4a3e-8af5-19affa7e1aa8"
+          (reference "RN8") (unit 4)
+        )
+      )
+    )
+  )
   (symbol (lib_id "power:GND") (at 152.4 107.95 0) (unit 1)
     (in_bom yes) (on_board yes) (dnp no)
@@
         )
       )
+    )
+  )
+  (symbol (lib_id "power:GND") (at 191.77 100.33 0) (unit 1)
+    (in_bom yes) (on_board yes) (dnp no)
+    (property "Reference" "#PWR0150" (at 191.77 106.68 0)
+      (effects (font (size 1.27 1.27)) hide)
+    )
+    (property "Value" "GND" (at 191.77 104.14 0)
+      (effects (font (size 1.27 1.27)))
+    )
+    (property "Footprint" "" (at 191.77 100.33 0)
+      (effects (font (size 1.27 1.27)) hide)
+    )
+    (property "Datasheet" "" (at 191.77 100.33 0)
+      (effects (font (size 1.27 1.27)) hide)
+    )
+    (pin "1")
+    (instances
+      (project "Revision 2"
+        (path "/3ba39048-ccb5-49b6-bc29-f9a8dd2e53b6/b80782fd-1148-4a3e-8af5-19affa7e1aa8"
+          (reference "#PWR0150") (unit 1)
+        )
+      )
+    )
+  )
+  (symbol (lib_id "Device:R_Pack04_Split") (at 185.42 82.55 270) (unit 1)
+    (in_bom yes) (on_board yes) (dnp no)
+    (property "Reference" "RN2" (at 185.4503 80.6009 90)
+      (effects (font (size 1.27 1.27)))
+    )
+    (property "Value" "10KΩ" (at 185.42 82.55 90)
+      (effects (font (size 1.27 1.27)))
+    )
+    (property "Footprint" "" (at 185.42 80.518 90)
+      (effects (font (size 1.27 1.27)) hide)
+    )
+    (property "Datasheet" "~" (at 185.42 82.55 0)
+      (effects (font (size 1.27 1.27)) hide)
+    )
+    (pin "1")
+    (pin "8")
+    (pin "2")
+    (pin "7")
+    (pin "3")
+    (pin "6")
+    (pin "4")
+    (pin "5")
+    (instances
+      (project "Revision 2"
+        (path "/3ba39048-ccb5-49b6-bc29-f9a8dd2e53b6/e0049583-c97a-4b82-a4d7-59c894eac2f8"
+          (reference "RN2") (unit 1)
+        )
+        (path "/3ba39048-ccb5-49b6-bc29-f9a8dd2e53b6/b80782fd-1148-4a3e-8af5-19affa7e1aa8"
+          (reference "RN8") (unit 1)
+        )
+      )
+    )
+  )
+  (symbol (lib_id "Device:R_Pack04_Split") (at 185.42 87.63 270) (unit 2)
+    (in_bom yes) (on_board yes) (dnp no)
+    (property "Reference" "RN2" (at 185.413 85.789 90)
+      (effects (font (size 1.27 1.27)))
+    )
+    (property "Value" "10KΩ" (at 185.42 87.63 90)
+      (effects (font (size 1.27 1.27)))
+    )
+    (property "Footprint" "" (at 185.42 85.598 90)
+      (effects (font (size 1.27 1.27)) hide)
+    )
+    (property "Datasheet" "~" (at 185.42 87.63 0)
+      (effects (font (size 1.27 1.27)) hide)
+    )
+    (pin "1")
+    (pin "8")
+    (pin "2")
+    (pin "7")
+    (pin "3")
+    (pin "6")
+    (pin "4")
+    (pin "5")
+    (instances
+      (project "Revision 2"
+        (path "/3ba39048-ccb5-49b6-bc29-f9a8dd2e53b6/e0049583-c97a-4b82-a4d7-59c894eac2f8"
+          (reference "RN2") (unit 2)
+        )
+        (path "/3ba39048-ccb5-49b6-bc29-f9a8dd2e53b6/b80782fd-1148-4a3e-8af5-19affa7e1aa8"
+          (reference "RN8") (unit 2)
+        )
+      )

Commit message: ESD protection diodes go BRRRRRRR
Parts:
- J4: now not fitted
Changed lines of the file:
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@@
   )
   (symbol (lib_id "Turaco:Conn_02x10_Odd_Even") (at 142.24 92.71 0) (unit 1)
-    (in_bom yes) (on_board yes) (dnp no)
+    (in_bom yes) (on_board yes) (dnp yes)
     (property "Reference" "J4" (at 142.24 80.01 0)
       (effects (font (size 1.27 1.27)))

Commit message: Updated re: issue #2
Parts:
- RN2: footprint (none) -> Resistor_SMD:R_Array_Concave_4x0402
Changed lines of the file:
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@@
     (effects (font (size 1.27 1.27)) (justify right bottom))
   )
-  (label "ETH_RX_CLK" (at 181.61 87.63 180)
+  (label "ETH_RX_CLK" (at 181.61 87.63 180) (fields_autoplaced)
     (effects (font (size 1.27 1.27)) (justify right bottom))
   )
@@
     (effects (font (size 1.27 1.27)) (justify right bottom))
   )
-  (label "ETH_COL" (at 181.61 92.71 180)
+  (label "ETH_COL" (at 181.61 92.71 180) (fields_autoplaced)
     (effects (font (size 1.27 1.27)) (justify right bottom))
   )
@@
     (effects (font (size 1.27 1.27)) (justify left bottom))
   )
-  (label "ETH_CRS" (at 181.61 82.55 180)
-    (effects (font (size 1.27 1.27)) (justify right bottom))
-  )
-  (label "ETH_TX_CLK" (at 181.61 97.79 180)
+  (label "ETH_CRS" (at 181.61 82.55 180) (fields_autoplaced)
+    (effects (font (size 1.27 1.27)) (justify right bottom))
+  )
+  (label "ETH_TX_CLK" (at 181.61 97.79 180) (fields_autoplaced)
     (effects (font (size 1.27 1.27)) (justify right bottom))
   )
@@
       (effects (font (size 1.27 1.27)))
     )
-    (property "Footprint" "" (at 185.42 90.678 90)
+    (property "Footprint" "Resistor_SMD:R_Array_Concave_4x0402" (at 185.42 90.678 90)
       (effects (font (size 1.27 1.27)) hide)
     )
@@
       (effects (font (size 1.27 1.27)))
     )
-    (property "Footprint" "" (at 185.42 95.758 90)
+    (property "Footprint" "Resistor_SMD:R_Array_Concave_4x0402" (at 185.42 95.758 90)
       (effects (font (size 1.27 1.27)) hide)
     )
@@
       (effects (font (size 1.27 1.27)))
     )
-    (property "Footprint" "" (at 185.42 80.518 90)
+    (property "Footprint" "Resistor_SMD:R_Array_Concave_4x0402" (at 185.42 80.518 90)
       (effects (font (size 1.27 1.27)) hide)
     )
@@
       (effects (font (size 1.27 1.27)))
     )
-    (property "Footprint" "" (at 185.42 85.598 90)
-      (effects (font (size 1.27 1.27)) hide)
-    )
+    (property "Footprint" "Resistor_SMD:R_Array_Concave_4x0402" (at 185.42 85.598 90)
+      (effects (font (size 1.27 1.27)) hide)
+    )
