File: PCB/Revision 2/ram.kicad_sch (KiCad schematic)
At the start: 3 parts, among them U6 AS7C38096A-10TIN

Commit message: Updated re: issue #2
Parts:
- C7: footprint (none) -> Capacitor_SMD:C_0402_1005Metric
Changed lines of the file:
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@@
       (effects (font (size 1.27 1.27)) (justify left))
     )
-    (property "Footprint" "" (at 160.9852 41.91 0)
+    (property "Footprint" "Capacitor_SMD:C_0402_1005Metric" (at 160.9852 41.91 0)
       (effects (font (size 1.27 1.27)) hide)
     )
@@
       (effects (font (size 1.27 1.27)) (justify left))
     )
-    (property "Footprint" "" (at 140.6652 41.91 0)
+    (property "Footprint" "Capacitor_SMD:C_0402_1005Metric" (at 140.6652 41.91 0)
       (effects (font (size 1.27 1.27)) hide)
     )
