File: PCB/Revision 2/usb_controller.kicad_sch (KiCad schematic)
At the start: 5 parts, among them U7 74LVC1G04

Commit message: Updated re: issue #2
Parts:
- added R3 (x2): 10Ω, symbol Device:R
- C36, C37, C38: footprint (none) -> Capacitor_SMD:C_0402_1005Metric
Connections:
- net RXD0: now also R3.1; no longer U8.13 (P2.7/TXD1)
- net TXD0: now also R3.1; no longer U8.12 (P2.6/RXD1)
- new net: R3.2, U8.12 (P2.6/RXD1)
- new net: R3.2, U8.13 (P2.7/TXD1)
Changed lines of the file:
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@@
   (no_connect (at 123.19 93.98))
   (no_connect (at 123.19 106.68))
-  (bus_entry (at 189.23 88.9) (size -2.54 2.54)
-    (stroke (width 0) (type default))
-  )
-  (bus_entry (at 189.23 91.44) (size -2.54 2.54)
+  (bus_entry (at 200.66 88.9) (size -2.54 2.54)
+    (stroke (width 0) (type default))
+  )
+  (bus_entry (at 200.66 91.44) (size -2.54 2.54)
     (stroke (width 0) (type default))
   )
@@
     (stroke (width 0) (type default))
   )
+  (wire (pts (xy 176.53 93.98) (xy 181.61 93.98))
+    (stroke (width 0) (type default))
+  )
   (bus (pts (xy 73.66 111.76) (xy 76.2 114.3))
     (stroke (width 0) (type default))
@@
     (stroke (width 0) (type default))
   )
-  (wire (pts (xy 176.53 93.98) (xy 186.69 93.98))
+  (wire (pts (xy 189.23 93.98) (xy 198.12 93.98))
+    (stroke (width 0) (type default))
+  )
+  (wire (pts (xy 176.53 91.44) (xy 181.61 91.44))
     (stroke (width 0) (type default))
   )
@@
     (stroke (width 0) (type default))
   )
-  (bus (pts (xy 189.23 86.36) (xy 191.77 83.82))
-    (stroke (width 0) (type default))
-  )
-  (bus (pts (xy 189.23 86.36) (xy 189.23 88.9))
-    (stroke (width 0) (type default))
-  )
-  (bus (pts (xy 189.23 88.9) (xy 189.23 91.44))
-    (stroke (width 0) (type default))
-  )
-  (wire (pts (xy 176.53 91.44) (xy 186.69 91.44))
+  (bus (pts (xy 200.66 86.36) (xy 203.2 83.82))
+    (stroke (width 0) (type default))
+  )
+  (wire (pts (xy 189.23 91.44) (xy 198.12 91.44))
+    (stroke (width 0) (type default))
+  )
+  (bus (pts (xy 200.66 86.36) (xy 200.66 88.9))
+    (stroke (width 0) (type default))
+  )
+  (bus (pts (xy 200.66 88.9) (xy 200.66 91.44))
     (stroke (width 0) (type default))
   )
@@
     (stroke (width 0) (type default))
   )
-  (bus (pts (xy 191.77 83.82) (xy 194.31 83.82))
+  (bus (pts (xy 203.2 83.82) (xy 205.74 83.82))
     (stroke (width 0) (type default))
   )
@@
     (stroke (width 0) (type default))
   )
-  (label "TXD0" (at 185.42 91.44 180) (fields_autoplaced)
+  (label "TXD0" (at 196.85 91.44 180) (fields_autoplaced)
     (effects (font (size 1.27 1.27)) (justify right bottom))
   )
@@
     (effects (font (size 1.27 1.27)) (justify left bottom))
   )
-  (label "RXD0" (at 185.42 93.98 180) (fields_autoplaced)
+  (label "RXD0" (at 196.85 93.98 180) (fields_autoplaced)
     (effects (font (size 1.27 1.27)) (justify right bottom))
   )
@@
     (effects (font (size 1.27 1.27)) (justify right))
   )
-  (hierarchical_label "{Serial Ports}" (shape bidirectional) (at 194.31 83.82 0) (fields_autoplaced)
+  (hierarchical_label "{Serial Ports}" (shape bidirectional) (at 205.74 83.82 0) (fields_autoplaced)
     (effects (font (size 1.27 1.27)) (justify left))
   )
@@
       (effects (font (size 1.27 1.27)) (justify left))
     )
-    (property "Footprint" "" (at 144.4752 73.66 0)
+    (property "Footprint" "Capacitor_SMD:C_0402_1005Metric" (at 144.4752 73.66 0)
       (effects (font (size 1.27 1.27)) hide)
     )
@@
       (effects (font (size 1.27 1.27)) (justify left))
     )
-    (property "Footprint" "" (at 166.0652 73.66 0)
+    (property "Footprint" "Capacitor_SMD:C_0402_1005Metric" (at 166.0652 73.66 0)
       (effects (font (size 1.27 1.27)) hide)
     )
@@
     )
   )
+  (symbol (lib_id "Device:R") (at 185.42 91.44 270) (unit 1)
+    (in_bom yes) (on_board yes) (dnp no)
+    (property "Reference" "R3" (at 185.42 88.9 90)
+      (effects (font (size 1.27 1.27)))
+    )
+    (property "Value" "10Ω" (at 185.42 91.44 90)
+      (effects (font (size 1.27 1.27)))
+    )
+    (property "Footprint" "" (at 185.42 89.662 90)
+      (effects (font (size 1.27 1.27)) hide)
+    )
+    (property "Datasheet" "~" (at 185.42 91.44 0)
+      (effects (font (size 1.27 1.27)) hide)
+    )
+    (pin "1")
+    (pin "2")
+    (instances
+      (project "Revision 2"
+        (path "/3ba39048-ccb5-49b6-bc29-f9a8dd2e53b6/ef7f0437-b22e-4c24-9273-d90d53267996"
+          (reference "R3") (unit 1)
+        )
+        (path "/3ba39048-ccb5-49b6-bc29-f9a8dd2e53b6/2f105b5f-8574-4519-9d4f-c6c87cbcfb0b"
+          (reference "R5") (unit 1)
+        )
+      )
+    )
+  )
   (symbol (lib_id "Turaco:C") (at 104.14 106.68 0) (unit 1)
     (in_bom yes) (on_board yes) (dnp no)
@@
       (effects (font (size 1.27 1.27)) (justify left))
     )
-    (property "Footprint" "" (at 105.1052 110.49 0)
+    (property "Footprint" "Capacitor_SMD:C_0402_1005Metric" (at 105.1052 110.49 0)
       (effects (font (size 1.27 1.27)) hide)
     )
@@
         )
       )
+    )
+  )
+  (symbol (lib_id "Device:R") (at 185.42 93.98 270) (unit 1)
+    (in_bom yes) (on_board yes) (dnp no)
+    (property "Reference" "R3" (at 185.42 96.52 90)
+      (effects (font (size 1.27 1.27)))
+    )
+    (property "Value" "10Ω" (at 185.42 93.98 90)
+      (effects (font (size 1.27 1.27)))
+    )
+    (property "Footprint" "" (at 185.42 92.202 90)
+      (effects (font (size 1.27 1.27)) hide)
+    )
+    (property "Datasheet" "~" (at 185.42 93.98 0)
+      (effects (font (size 1.27 1.27)) hide)
+    )
+    (pin "1")
+    (pin "2")
+    (instances
+      (project "Revision 2"
+        (path "/3ba39048-ccb5-49b6-bc29-f9a8dd2e53b6/ef7f0437-b22e-4c24-9273-d90d53267996"
+          (reference "R3") (unit 1)
+        )
+        (path "/3ba39048-ccb5-49b6-bc29-f9a8dd2e53b6/2f105b5f-8574-4519-9d4f-c6c87cbcfb0b"
+          (reference "R6") (unit 1)
+        )
+      )
